Commit message: add collision information on gripper

File: depowdering_aman/urdf/depowdering_gripper_robot.xacro (robot description, xacro)
@@ -269,10 +269,10 @@
 			</material>
 		</visual>
-		<!-- <collision>
-			<origin xyz="0 0 0" rpy="0 0 0" />
+		<collision>
+			<origin xyz="0 0 -0.05" rpy="0 0 0" />
 			<geometry>
 				<mesh filename="package://add_post_pro_simulation/mesh/gripper_Link.STL" />
 			</geometry>
-		</collision> -->
+		</collision>
 	</link>
 	<joint name="gripper_base_Joint" type="fixed">
